File: circuit/PWM3ch.sch (KiCad schematic (older format))
At the start: 26 parts

Commit message: schematic: HSV operation and power from ICSP.
Parts:
- removed RV?: BLUE, symbol POT
- added JP1: Jumper_NO_Small, symbol Jumper_NO_Small
- RV1: renamed from RV?; value BRIGHT -> HUE
- RV2: renamed from RV?; value RED -> SAT
- RV3: renamed from RV?; value GREEN -> VAL
- gave numbers to parts that had none: 22
Connections:
- net GND: now also RV1.3, RV2.3, RV3.3; no longer RV1.1, RV2.1, RV3.1
- net VCC: now also RV1.1, RV2.1, RV3.1, JP1.2; no longer RV1.3, RV2.3, RV3.3
- net at IC1.10 ((PCINT3/T0/ADC3)PA3): now also Q1.2 (B)
- net at IC1.7 ((PCINT6/SDA/DI/MOSI/OC1A/ADC6)PA6), P2.4 (P4): no longer Q1.2 (B)
- net at P2.2 (P2): now also JP1.1
- no-connect marks 1 -> 0
Other:
- note added: "OPTIONAL: a jumper to allow\npowering from ICSP."
